File: CAMERA.kicad_pcb (KiCad board)
At the start: 6 copper layers, 88 parts, among them J1 Conn_01x06_Male, J10 E, J11 F, J12 G, J13 H, J14 J, J15 K, J16 L, J17 M, J18 N, J19 P, J2 Conn_01x08_Male, J20 R, J21 T, J22 Conn_01x10_Male, J23 Conn_01x08_Male, J26 Conn_01x25_Pin, J27 Conn_01x25_Pin, J28 Conn_01x25_Pin, J29 Conn_01x25_Pin, J3 A, J4 U, J5 B, J6 V, J7 C, J8 W, J9 D, Q1 BC550

Commit message: Add files via upload
Other:
- board text added: "Picot en bas à gauche en vue de dessus Gestion d'un capteur d'image MT9M413 Version 2, 12/04/2025, Edern Ollivier"
- board text removed: "Picot en bas à gauche en vue de dessus Gestion d'un capteur d'image MT9M413 Version 2, 18/04/2025, Edern Ollivier"
Changed lines of the file:
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@@
 	)
 	(gr_rect
-		(start 17.78 20.32)
-		(end 274.32 142.24)
+		(start 17.78 25.4)
+		(end 274.32 137.16)
 		(stroke
 			(width 0.2)
@@
 		)
 	)
-	(gr_text "Picot en bas à gauche en vue de dessus\nGestion d'un capteur d'image MT9M413\nVersion 2, 18/04/2025, Edern Ollivier\n"
+	(gr_text "Picot en bas à gauche en vue de dessus\nGestion d'un capteur d'image MT9M413\nVersion 2, 12/04/2025, Edern Ollivier\n"
 		(at 121.92 33.02 0)
 		(layer "F.SilkS")
@@
 		(polygon
 			(pts
-				(xy 274.32 20.32) (xy 274.32 142.24) (xy 17.78 142.24) (xy 17.78 20.32)
+				(xy 274.32 25.4) (xy 274.32 137.16) (xy 17.78 137.16) (xy 17.78 25.4)
 			)
 		)
